File: JAT 3t amplifier.sch (KiCad schematic (older format))
At the start: 19 parts, among them Q1 2n2222, Q2 2n2222, Q3 2n2907

Commit message: Add files via upload
Parts:
- C1: footprint (none) -> Capacitor_THT:CP_Radial_Tantal_D6.0mm_P5.00mm
- C2, C3, C4: footprint (none) -> Capacitor_THT:CP_Radial_D6.3mm_P2.50mm
- C5: footprint (none) -> Capacitor_THT:CP_Radial_D8.0mm_P2.50mm
- D1, D2: footprint (none) -> Diode_THT:D_DO-41_SOD81_P7.62mm_Horizontal
- Q1, Q2, Q3: footprint (none) -> Package_TO_SOT_THT:TO-92
- R1, R2, R3, R4, R5, R6, R7: footprint (none) -> Resistor_THT:R_Axial_DIN0207_L6.3mm_D2.5mm_P7.62mm_Horizontal
- RV1, RV2: footprint (none) -> Potentiometer_THT:Potentiometer_ACP_CA9-H5_Horizontal
Changed lines of the file:
@@
 F 0 "C2" V 3502 6250 50  0000 C CNN
 F 1 "47u" V 3411 6250 50  0000 C CNN
-F 2 "" H 3288 6100 50  0001 C CNN
+F 2 "Capacitor_THT:CP_Radial_D6.3mm_P2.50mm" H 3288 6100 50  0001 C CNN
 F 3 "~" H 3250 6250 50  0001 C CNN
 	1    3250 6250
@@
 F 0 "RV1" H 3632 6204 50  0000 R CNN
 F 1 "5k" H 3632 6295 50  0000 R CNN
-F 2 "" H 3700 6250 50  0001 C CNN
+F 2 "Potentiometer_THT:Potentiometer_ACP_CA9-H5_Horizontal" H 3700 6250 50  0001 C CNN
 F 3 "~" H 3700 6250 50  0001 C CNN
 	1    3700 6250
@@
 F 0 "R3" H 4218 6296 50  0000 L CNN
 F 1 "4.7k" H 4218 6205 50  0000 L CNN
-F 2 "" V 4190 6240 50  0001 C CNN
+F 2 "Resistor_THT:R_Axial_DIN0207_L6.3mm_D2.5mm_P7.62mm_Horizontal" V 4190 6240 50  0001 C CNN
 F 3 "~" H 4150 6250 50  0001 C CNN
 	1    4150 6250
@@
 F 0 "RV2" H 4082 5496 50  0000 R CNN
 F 1 "20k" H 4082 5405 50  0000 R CNN
-F 2 "" H 4150 5450 50  0001 C CNN
+F 2 "Potentiometer_THT:Potentiometer_ACP_CA9-H5_Horizontal" H 4150 5450 50  0001 C CNN
 F 3 "~" H 4150 5450 50  0001 C CNN
 	1    4150 5450
@@
 F 0 "Q2" H 5241 4296 50  0000 L CNN
 F 1 "2n2222" H 5241 4205 50  0000 L CNN
-F 2 "" H 5250 4350 50  0001 C CNN
+F 2 "Package_TO_SOT_THT:TO-92" H 5250 4350 50  0001 C CNN
 F 3 "~" H 5050 4250 50  0001 C CNN
 	1    5050 4250
@@
 F 0 "Q3" H 5241 5646 50  0000 L CNN
 F 1 "2n2907" H 5241 5555 50  0000 L CNN
-F 2 "" H 5250 5700 50  0001 C CNN
+F 2 "Package_TO_SOT_THT:TO-92" H 5250 5700 50  0001 C CNN
 F 3 "~" H 5050 5600 50  0001 C CNN
 	1    5050 5600
@@
 F 0 "Q1" H 4741 5996 50  0000 L CNN
 F 1 "2n2222" H 4741 5905 50  0000 L CNN
-F 2 "" H 4750 6050 50  0001 C CNN
+F 2 "Package_TO_SOT_THT:TO-92" H 4750 6050 50  0001 C CNN
 F 3 "~" H 4550 5950 50  0001 C CNN
 	1    4550 5950
@@
 F 0 "D2" V 4696 5071 50  0000 R CNN
 F 1 "1n4007" V 4605 5071 50  0000 R CNN
-F 2 "" H 4650 5150 50  0001 C CNN
+F 2 "Diode_THT:D_DO-41_SOD81_P7.62mm_Horizontal" H 4650 5150 50  0001 C CNN
 F 3 "~" H 4650 5150 50  0001 C CNN
 	1    4650 5150
@@
 F 0 "D1" V 4696 4571 50  0000 R CNN
 F 1 "1n4007" V 4605 4571 50  0000 R CNN
-F 2 "" H 4650 4650 50  0001 C CNN
+F 2 "Diode_THT:D_DO-41_SOD81_P7.62mm_Horizontal" H 4650 4650 50  0001 C CNN
 F 3 "~" H 4650 4650 50  0001 C CNN
 	1    4650 4650
@@
 F 0 "R6" H 5218 4696 50  0000 L CNN
 F 1 ".47" H 5218 4605 50  0000 L CNN
-F 2 "" V 5190 4640 50  0001 C CNN
+F 2 "Resistor_THT:R_Axial_DIN0207_L6.3mm_D2.5mm_P7.62mm_Horizontal" V 5190 4640 50  0001 C CNN
 F 3 "~" H 5150 4650 50  0001 C CNN
 	1    5150 4650
@@
 F 0 "R7" H 5218 5196 50  0000 L CNN
 F 1 ".47" H 5218 5105 50  0000 L CNN
-F 2 "" V 5190 5140 50  0001 C CNN
+F 2 "Resistor_THT:R_Axial_DIN0207_L6.3mm_D2.5mm_P7.62mm_Horizontal" V 5190 5140 50  0001 C CNN
 F 3 "~" H 5150 5150 50  0001 C CNN
 	1    5150 5150
@@
 F 0 "C5" V 5902 4900 50  0000 C CNN
 F 1 "470u" V 5811 4900 50  0000 C CNN
-F 2 "" H 5650 4900 50  0001 C CNN
+F 2 "Capacitor_THT:CP_Radial_D8.0mm_P2.50mm" H 5650 4900 50  0001 C CNN
 F 3 "~" H 5650 4900 50  0001 C CNN
 	1    5650 4900
@@
 F 0 "C3" H 4265 4346 50  0000 L CNN
 F 1 "100u" H 4265 4255 50  0000 L CNN
-F 2 "" H 4150 4300 50  0001 C CNN
+F 2 "Capacitor_THT:CP_Radial_D6.3mm_P2.50mm" H 4150 4300 50  0001 C CNN
 F 3 "~" H 4150 4300 50  0001 C CNN
 	1    4150 4300
@@
 F 0 "R5" H 4718 4046 50  0000 L CNN
 F 1 "470" H 4718 3955 50  0000 L CNN
-F 2 "" V 4690 3990 50  0001 C CNN
+F 2 "Resistor_THT:R_Axial_DIN0207_L6.3mm_D2.5mm_P7.62mm_Horizontal" V 4690 3990 50  0001 C CNN
 F 3 "~" H 4650 4000 50  0001 C CNN
 	1    4650 4000
@@
 F 0 "R4" H 4718 3496 50  0000 L CNN
 F 1 "470" H 4718 3405 50  0000 L CNN
-F 2 "" V 4690 3440 50  0001 C CNN
+F 2 "Resistor_THT:R_Axial_DIN0207_L6.3mm_D2.5mm_P7.62mm_Horizontal" V 4690 3440 50  0001 C CNN
 F 3 "~" H 4650 3450 50  0001 C CNN
 	1    4650 3450
@@
 F 0 "C4" H 5715 3496 50  0000 L CNN
 F 1 "100u" H 5715 3405 50  0000 L CNN
-F 2 "" H 5600 3450 50  0001 C CNN
+F 2 "Capacitor_THT:CP_Radial_D6.3mm_P2.50mm" H 5600 3450 50  0001 C CNN
 F 3 "~" H 5600 3450 50  0001 C CNN
 	1    5600 3450
@@
 F 0 "R1" V 1995 6250 50  0000 C CNN
 F 1 "220" V 2086 6250 50  0000 C CNN
-F 2 "" V 2240 6240 50  0001 C CNN
+F 2 "Resistor_THT:R_Axial_DIN0207_L6.3mm_D2.5mm_P7.62mm_Horizontal" V 2240 6240 50  0001 C CNN
 F 3 "~" H 2200 6250 50  0001 C CNN
 	1    2200 6250
@@
 F 0 "C1" H 2615 6646 50  0000 L CNN
 F 1 "100n" H 2615 6555 50  0000 L CNN
-F 2 "" H 2538 6450 50  0001 C CNN
+F 2 "Capacitor_THT:CP_Radial_Tantal_D6.0mm_P5.00mm" H 2538 6450 50  0001 C CNN
 F 3 "~" H 2500 6600 50  0001 C CNN
 	1    2500 6600
@@
 F 0 "R2" H 2832 6554 50  0000 R CNN
 F 1 "100" H 2832 6645 50  0000 R CNN
-F 2 "" V 2940 6590 50  0001 C CNN
+F 2 "Resistor_THT:R_Axial_DIN0207_L6.3mm_D2.5mm_P7.62mm_Horizontal" V 2940 6590 50  0001 C CNN
 F 3 "~" H 2900 6600 50  0001 C CNN
 	1    2900 6600
